Commit message: added rgb-d cam plugin

File: diff_description/urdf/robot.xacro (robot description, xacro)
@@ -49,33 +49,59 @@
     </visual>
   </link>
-<xacro:link_wheel name="link_right_wheel" />
-<xacro:joint_wheel name="joint_right_wheel" child="link_right_wheel" origin_xyz="-0.05 -0.15 0"/>
-<xacro:link_wheel name="link_left_wheel" />
-<xacro:joint_wheel name="joint_left_wheel" child="link_left_wheel" origin_xyz="-0.05 0.15 0"/>
-<link name="sensor_laser">
-  <inertial>
-    <origin xyz="0 0 0" rpy="0 0 0" />
-    <mass value="1" />
-    <!-- RANDOM INERTIA BELOW -->
-    <inertia ixx="0.02" ixy="0" ixz="0" iyy="0.02" iyz="0" izz="0.02"/>
-  </inertial>
-  <visual>
-    <origin xyz="0 0 0" rpy="0 0 0" />
-    <geometry>
-      <cylinder radius="0.05" length="0.1"/>
-    </geometry>
-    <material name="white" />
-  </visual>
-  <collision>
-    <origin xyz="0 0 0" rpy="0 0 0"/>
-    <geometry>
-      <cylinder radius="0.05" length="0.1"/>
-    </geometry>
-  </collision>
-</link>
-<joint name="joint_sensor_laser" type="fixed">
-  <origin xyz="0.15 0 0.05" rpy="0 0 0"/>
-  <parent link="link_chassis"/>
-  <child link="sensor_laser"/>
-</joint>
+  <xacro:link_wheel name="link_right_wheel" />
+  <xacro:joint_wheel name="joint_right_wheel" child="link_right_wheel" origin_xyz="-0.05 -0.15 0"/>
+  <xacro:link_wheel name="link_left_wheel" />
+  <xacro:joint_wheel name="joint_left_wheel" child="link_left_wheel" origin_xyz="-0.05 0.15 0"/>
+  <link name="sensor_laser">
+    <inertial>
+      <origin xyz="0 0 0" rpy="0 0 0" />
+      <mass value="1" />
+      <!-- RANDOM INERTIA BELOW -->
+      <inertia ixx="0.02" ixy="0" ixz="0" iyy="0.02" iyz="0" izz="0.02"/>
+    </inertial>
+    <visual>
+      <origin xyz="0 0 0" rpy="0 0 0" />
+      <geometry>
+        <cylinder radius="0.05" length="0.1"/>
+      </geometry>
+      <material name="white" />
+    </visual>
+    <collision>
+      <origin xyz="0 0 0" rpy="0 0 0"/>
+      <geometry>
+        <cylinder radius="0.05" length="0.1"/>
+      </geometry>
+    </collision>
+  </link>
+  <link name="kinect_sensor">
+    <inertial>
+      <origin xyz="0 0 0" rpy="0 0 0" />
+      <mass value="1" />
+      <!-- RANDOM INERTIA BELOW -->
+      <inertia ixx="0.02" ixy="0" ixz="0" iyy="0.02" iyz="0" izz="0.02"/>
+    </inertial>
+    <visual>
+      <origin xyz="0 0 0" rpy="0 0 0" />
+      <geometry>
+        <box size="0.1 0.15 0.1"/>
+      </geometry>
+      <material name="red" />
+    </visual>
+    <collision>
+      <origin xyz="0 0 0" rpy="0 0 0"/>
+      <geometry>
+        <box size="0.1 0.15 0.1"/>
+      </geometry>
+    </collision>
+  </link>
+  <joint name="joint_sensor_laser" type="fixed">
+    <origin xyz="0 0 0.1" rpy="0 0 0"/>
+    <parent link="kinect_sensor"/>
+    <child link="sensor_laser"/>
+  </joint>
+  <joint name="joint_sensor_kinect" type="fixed">
+    <origin xyz="0.15 0 0.1" rpy="0 0 0"/>
+    <parent link="link_chassis"/>
+    <child link="kinect_sensor"/>
+  </joint>
 </robot>
